File: Hardware_electronic/kicad/e256_teensy4_0/e256_teensy4_0.kicad_pcb (KiCad board)
At the start: 2 copper layers, 76 x 70 mm, 58 parts, among them J0 Conn_Coaxial_Power, J1 MIDI_IN, J2 MIDI_OUT, J3 AUDIO_IN, J4 AUDIO_OUT, J5 LINE_OUT, J6 e256_pad_16x16, SW1 SW_Push, SW2 SW_Push, SW3 RotaryEncoder_Switch, U1 6N138SM, U10 W25Q128JVS, U2 Teensy4.0, U3 74HC595BQ, U4 74HC595BQ, U5 74HC595BQ, U6 74HC4051BQ, U7 74HC4051BQ, U8 MCP1811A, U9 SGTL5000

Commit message: Fix: clear llist_mappings before applying new config to prevent duplicates
- Clear llist_mappings at the start of mappings_load_config so repeated
  UPLOAD→APPLY cycles don't accumulate duplicate mapping entries; each
  llist_pop_front returns the node to the pool (no memory leak)
- Add turnThruOff() and while(HARDWARE_MIDI.read()) to fix hardware MIDI
  IN callback not triggering when a keyboard is connected
- Various firmware and hardware updates

Co-Authored-By: Claude Sonnet 4.6 <noreply@anthropic.com>
Other:
- net class +5V removed
- net class AUDIO_OUT removed
- net class Default removed
- net class GND removed
- net class VCC removed
